Commit message: updated demo to park at the parking spot (basic)

File: gem_simulator/gem_description/urdf/gem_e4.urdf.xacro (robot description, xacro)
@@ -46,5 +46,5 @@
     <material>Gazebo/Blue</material>
   </gazebo>
-  <joint name="base_link" type="fixed">
+  <joint name="base_footprint_to_base_link" type="fixed">
     <origin xyz="0 0 0.268" rpy="0 0 0" />
     <parent link="base_footprint" />
